File: Motorcycle/smart_helmet/smart_helmet.kicad_sch (KiCad schematic)
At the start: 6 parts, among them U2 TSL2561, U3 LM340K-5.0/NOPB, U4 LP2950-3.3_TO252, U5 ESP32-WROOM-32

Commit message: first draft PCB done
Parts:
- R1, R2: footprint (none) -> Resistor_SMD:R_0805_2012Metric_Pad1.20x1.40mm_HandSolder
- U3: footprint K02A_TEX -> footprints:LM340K-5.0&slash_NOPB
Changed lines of the file:
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@@
       (effects (font (size 1.524 1.524)))
     )
-    (property "Footprint" "K02A_TEX" (at 143.51 31.75 0)
+    (property "Footprint" "footprints:LM340K-5.0&slash_NOPB" (at 143.51 31.75 0)
       (effects (font (size 1.27 1.27) italic) hide)
     )
@@
       (effects (font (size 1.27 1.27)) (justify left))
     )
-    (property "Footprint" "" (at 99.822 83.82 90)
+    (property "Footprint" "Resistor_SMD:R_0805_2012Metric_Pad1.20x1.40mm_HandSolder" (at 99.822 83.82 90)
       (effects (font (size 1.27 1.27)) hide)
     )
@@
       (effects (font (size 1.27 1.27)) (justify left))
     )
-    (property "Footprint" "" (at 107.442 87.63 90)
-      (effects (font (size 1.27 1.27)) hide)
-    )
+    (property "Footprint" "Resistor_SMD:R_0805_2012Metric_Pad1.20x1.40mm_HandSolder" (at 107.442 87.63 90)
+      (effects (font (size 1.27 1.27)) hide)
+    )
